File: PCB.kicad_pcb (KiCad board)
At the start: 2 copper layers, 89 x 160.1 mm, 42 parts, among them U1 WeMos_D1_mini

Commit message: generovany gerbery z projektu
Parts:
- removed H10, H11: MountingHole, MountingHole:MountingHole_3mm
- removed H9: MountingHole, MountingHole:MountingHole_4mm
- removed U1: WeMos_D1_mini, Module:WEMOS_D1_mini_light
- added G***: LOGO, LOGO, B.Cu at (116.7, 98.3)
- added H3: MountingHole, MountingHole:MountingHole_3mm, B.Cu at (142.9, 66.7)
- added H4: MountingHole, MountingHole:MountingHole_4mm, B.Cu at (82.5, 158.1)
- added H5: MountingHole, MountingHole:MountingHole_3mm, B.Cu at (65.4, 66.7)
- added U_WeMos_D1_Mini_Pro_1: WeMos_D1_Mini_Pro, Module:WEMOS_D1_mini_light, F.Cu at (91.3, 117.7)
Other:
- board text added: "Honeywell Intelligrated ------------------------- Project: ME commissioning of conveyors with VFDs controllable using digital outputs PCB Version: v 1.0. Creator: David Strasak"
